File: Design/nRF_Breakout.sch (KiCad schematic (older format))
At the start: 14 parts, among them IC1 LM1117, P1 CONN_01X18, P10 CONN_01X01, P2 CONN_01X08, P3 CONN_01X18, P5 CONN_01X08, P7 CONN_01X01, P8 CONN_01X01, P9 CONN_01X01, U1 nRF51822

Commit message: ADDED NEW FILES
Parts:
- added C1: 10uF, symbol CP1
- added C2: 0.1uF, symbol C
- added P4: CONN_01X02, symbol CONN_01X02
Connections:
- net GND: now also C1.2, C2.2, P4.1 (P1)
- net at IC1.3 (IN): now also C1.1, P4.2 (P2)
- net +3.3VP: no longer names the net of IC1.2 (OUT), IC1.4 (OUT), P1.11 (P11), R2.1, U1.11
- net +3.3VP: now also C2.1
- net ST_LED: no longer names the net of P1.2 (P2), R1.1, U1.2
- no-connect marks 21 -> 20
Other:
- moved on the sheet: D1, D2, IC1, P10, P7, P8, P9, R1, R2

Commit message: Corrected File
Parts:
- removed D2: LED, symbol LED
- removed P10, P9: CONN_01X01, symbol CONN_01X01
- removed R2: 470r, symbol R
- added P6: CONN_01X02, symbol CONN_01X02
Connections:
- net at P3.6 (P6), U1.31: now also P6.2 (P2)
- net at P3.5 (P5), U1.32: now also P6.1 (P1)
- no-connect marks 20 -> 18
Other:
- moved on the sheet: P7, P8
Changed lines of the file:
@@
 L CONN_01X01 P7
 U 1 1 55CB50F6
-P 6650 1100
-F 0 "P7" H 6650 1200 50  0000 C CNN
-F 1 "CONN_01X01" V 6750 1100 50  0000 C CNN
-F 2 "" H 6650 1100 60  0000 C CNN
-F 3 "" H 6650 1100 60  0000 C CNN
-	1    6650 1100
-	1    0    0    -1
-$EndComp
-$Comp
-L CONN_01X01 P9
-U 1 1 55CB52A5
-P 7200 1100
-F 0 "P9" H 7200 1200 50  0000 C CNN
-F 1 "CONN_01X01" V 7300 1100 50  0000 C CNN
-F 2 "" H 7200 1100 60  0000 C CNN
-F 3 "" H 7200 1100 60  0000 C CNN
-	1    7200 1100
-	1    0    0    -1
-$EndComp
-$Comp
-L CONN_01X01 P10
-U 1 1 55CB52EB
-P 7200 1750
-F 0 "P10" H 7200 1850 50  0000 C CNN
-F 1 "CONN_01X01" V 7300 1750 50  0000 C CNN
-F 2 "" H 7200 1750 60  0000 C CNN
-F 3 "" H 7200 1750 60  0000 C CNN
-	1    7200 1750
+P 7200 1050
+F 0 "P7" H 7200 1150 50  0000 C CNN
+F 1 "CONN_01X01" V 7300 1050 50  0000 C CNN
+F 2 "" H 7200 1050 60  0000 C CNN
+F 3 "" H 7200 1050 60  0000 C CNN
+	1    7200 1050
 	1    0    0    -1
 $EndComp
@@
 L CONN_01X01 P8
 U 1 1 55CB5314
-P 6650 1750
-F 0 "P8" H 6650 1850 50  0000 C CNN
-F 1 "CONN_01X01" V 6750 1750 50  0000 C CNN
-F 2 "" H 6650 1750 60  0000 C CNN
-F 3 "" H 6650 1750 60  0000 C CNN
-	1    6650 1750
-	1    0    0    -1
-$EndComp
-NoConn ~ 7000 1100
-NoConn ~ 7000 1750
-NoConn ~ 6450 1100
-NoConn ~ 6450 1750
+P 7200 1600
+F 0 "P8" H 7200 1700 50  0000 C CNN
+F 1 "CONN_01X01" V 7300 1600 50  0000 C CNN
+F 2 "" H 7200 1600 60  0000 C CNN
+F 3 "" H 7200 1600 60  0000 C CNN
+	1    7200 1600
+	1    0    0    -1
+$EndComp
+NoConn ~ 7000 1050
+NoConn ~ 7000 1600
 NoConn ~ 4350 3000
 NoConn ~ 4350 3100
@@
 	1950 1050 1950 1000
 $Comp
-L GND #PWR02
+L GND #PWR1
 U 1 1 55CB575A
 P 1650 2050
-F 0 "#PWR02" H 1650 1800 60  0001 C CNN
+F 0 "#PWR1" H 1650 1800 60  0001 C CNN
 F 1 "GND" H 1650 1900 60  0000 C CNN
 F 2 "" H 1650 2050 60  0000 C CNN
@@
 Wire Wire Line
 	1650 1300 1650 2050
-$Comp
-L LED D2
-U 1 1 55CB6D6E
-P 2600 1800
-F 0 "D2" H 2600 1900 50  0000 C CNN
-F 1 "LED" H 2600 1700 50  0000 C CNN
-F 2 "" H 2600 1800 60  0000 C CNN
-F 3 "" H 2600 1800 60  0000 C CNN
-	1    2600 1800
-	0    1    1    0
-$EndComp
-$Comp
-L R R2
-U 1 1 55CB6DC1
-P 2600 1300
-F 0 "R2" V 2680 1300 50  0000 C CNN
-F 1 "470r" V 2607 1301 50  0000 C CNN
-F 2 "" V 2530 1300 30  0000 C CNN
-F 3 "" H 2600 1300 30  0000 C CNN
-	1    2600 1300
-	1    0    0    -1
-$EndComp
-Wire Wire Line
-	2600 2000 2600 2050
-Wire Wire Line
-	2600 1600 2600 1550
 $Comp
 L nRF51822 U1
@@
 	5500 1250 5800 1250
 Wire Wire Line
-	5500 1350 5800 1350
-Wire Wire Line
-	5500 1450 5800 1450
+	5500 1350 6150 1350
+Wire Wire Line
+	5500 1450 6150 1450
 Wire Wire Line
 	5500 1550 5800 1550
@@
 Wire Wire Line
 	1950 1000 3650 1000
-Wire Wire Line
-	2600 1000 2600 1050
-Connection ~ 2600 1000
 Connection ~ 3300 2050
-Connection ~ 2600 2050
 Connection ~ 3750 2050
+$Comp
+L CONN_01X02 P6
+U 1 1 55D423AE
+P 6350 1400
+F 0 "P6" H 6350 1550 50  0000 C CNN
+F 1 "CONN_01X02" V 6450 1400 50  0000 C CNN
+F 2 "" H 6350 1400 60  0000 C CNN
+F 3 "" H 6350 1400 60  0000 C CNN
+	1    6350 1400
+	1    0    0    -1
+$EndComp
+Connection ~ 5800 1350
+Connection ~ 5800 1450
 $EndSCHEMATC

Commit message: Changed name
Connections:
- net at U1.34: now also P3.2 (P2); no longer P3.3 (P3)
- net at U1.35: now also P3.3 (P3); no longer P3.2 (P2)
Changed lines of the file:
@@
 	1    0    0    -1
 $EndComp
-Wire Wire Line
-	3300 1550 3300 1600
-Wire Wire Line
-	3300 2000 3300 2050
 $Comp
 L LM1117 IC1
@@
 NoConn ~ 5800 3600
 NoConn ~ 5800 3700
-Wire Wire Line
-	1950 1050 1950 1000
-$Comp
-L GND #PWR1
+$Comp
+L GND #PWR01
 U 1 1 55CB575A
 P 1650 2050
-F 0 "#PWR1" H 1650 1800 60  0001 C CNN
+F 0 "#PWR01" H 1650 1800 60  0001 C CNN
 F 1 "GND" H 1650 1900 60  0000 C CNN
 F 2 "" H 1650 2050 60  0000 C CNN
@@
 	1    0    0    -1
 $EndComp
-Wire Wire Line
-	1650 1300 1650 2050
 $Comp
 L nRF51822 U1
@@
 	1    0    0    -1
 $EndComp
-Wire Wire Line
-	3750 950  4700 950
-Wire Wire Line
-	3300 1050 4700 1050
-Wire Wire Line
-	4350 1150 4700 1150
-Wire Wire Line
-	4350 1250 4700 1250
-Wire Wire Line
-	4350 1350 4700 1350
-Wire Wire Line
-	4350 1450 4700 1450
-Wire Wire Line
-	4350 1550 4700 1550
-Wire Wire Line
-	4350 1650 4700 1650
-Wire Wire Line
-	4350 1750 4700 1750
-Wire Wire Line
-	4350 1850 4700 1850
-Wire Wire Line
-	3650 1950 4700 1950
-Wire Wire Line
-	1650 2050 4700 2050
-Wire Wire Line
-	4350 2150 4700 2150
-Wire Wire Line
-	4350 2250 4700 2250
-Wire Wire Line
-	4350 2350 4700 2350
-Wire Wire Line
-	4350 2450 4700 2450
-Wire Wire Line
-	4350 2550 4700 2550
-Wire Wire Line
-	4350 2650 4700 2650
-Wire Wire Line
-	5500 950  5800 950
-Wire Wire Line
-	5500 1050 5800 1050
-Wire Wire Line
-	5500 1150 5800 1150
-Wire Wire Line
-	5500 1250 5800 1250
-Wire Wire Line
-	5500 1350 6150 1350
-Wire Wire Line
-	5500 1450 6150 1450
-Wire Wire Line
-	5500 1550 5800 1550
-Wire Wire Line
-	5500 1650 5800 1650
-Wire Wire Line
-	5500 1750 5800 1750
-Wire Wire Line
-	5500 1850 5800 1850
-Wire Wire Line
-	5500 1950 5800 1950
-Wire Wire Line
-	5500 2050 5800 2050
-Wire Wire Line
-	5500 2150 5800 2150
-Wire Wire Line
-	5500 2250 5800 2250
-Wire Wire Line
-	5500 2350 5800 2350
-Wire Wire Line
-	5500 2450 5800 2450
-Wire Wire Line
-	5500 2550 5800 2550
-Wire Wire Line
-	5500 2650 5800 2650
-Wire Wire Line
-	3750 950  3750 2050
-Connection ~ 4350 950
-Wire Wire Line
-	3650 1000 3650 1950
-Connection ~ 4350 1950
-Connection ~ 4350 2050
 $Comp
 L CONN_01X02 P4
@@
 	-1   0    0    1
 $EndComp
-Wire Wire Line
-	1100 1100 1100 1450
 $Comp
 L CP1 C1
@@
 	1    0    0    -1
 $EndComp
-Wire Wire Line
-	1100 1000 1350 1000
-Wire Wire Line
-	1250 1050 1250 1000
-Connection ~ 1250 1000
-Wire Wire Line
-	1100 1450 2050 1450
-Connection ~ 1250 1450
-Connection ~ 1650 1450
-Wire Wire Line
-	2050 1050 2050 1000
-Connection ~ 2050 1000
 $Comp
 L C C2
@@
 	1    0    0    -1
 $EndComp
-Connection ~ 4350 1050
-Wire Wire Line
-	1950 1000 3650 1000
-Connection ~ 3300 2050
-Connection ~ 3750 2050
 $Comp
 L CONN_01X02 P6
@@
 	1    0    0    -1
 $EndComp
+Wire Wire Line
+	3300 1550 3300 1600
+Wire Wire Line
+	3300 2000 3300 2050
+Wire Wire Line
+	1950 1050 1950 1000
+Wire Wire Line
+	1650 1300 1650 2050
+Wire Wire Line
+	3750 950  4700 950
+Wire Wire Line
+	3300 1050 4700 1050
+Wire Wire Line
+	4350 1150 4700 1150
+Wire Wire Line
+	4350 1250 4700 1250
+Wire Wire Line
+	4350 1350 4700 1350
+Wire Wire Line
+	4350 1450 4700 1450
+Wire Wire Line
+	4350 1550 4700 1550
+Wire Wire Line
+	4350 1650 4700 1650
+Wire Wire Line
+	4350 1750 4700 1750
+Wire Wire Line
+	4350 1850 4700 1850
+Wire Wire Line
+	3650 1950 4700 1950
+Wire Wire Line
+	1650 2050 4700 2050
+Wire Wire Line
+	4350 2150 4700 2150
+Wire Wire Line
+	4350 2250 4700 2250
+Wire Wire Line
+	4350 2350 4700 2350
+Wire Wire Line
+	4350 2450 4700 2450
+Wire Wire Line
+	4350 2550 4700 2550
+Wire Wire Line
+	4350 2650 4700 2650
+Wire Wire Line
+	5500 950  5800 950
+Wire Wire Line
+	5500 1250 5800 1250
+Wire Wire Line
+	5500 1350 6150 1350
+Wire Wire Line
+	5500 1450 6150 1450
+Wire Wire Line
+	5500 1550 5800 1550
+Wire Wire Line
+	5500 1650 5800 1650
+Wire Wire Line
+	5500 1750 5800 1750
+Wire Wire Line
+	5500 1850 5800 1850
+Wire Wire Line
+	5500 1950 5800 1950
+Wire Wire Line
+	5500 2050 5800 2050
+Wire Wire Line
+	5500 2150 5800 2150
+Wire Wire Line
+	5500 2250 5800 2250
+Wire Wire Line
+	5500 2350 5800 2350
+Wire Wire Line
+	5500 2450 5800 2450
+Wire Wire Line
+	5500 2550 5800 2550
+Wire Wire Line
+	5500 2650 5800 2650
+Wire Wire Line
+	3750 950  3750 2050
+Connection ~ 4350 950
+Wire Wire Line
+	3650 1000 3650 1950
+Connection ~ 4350 1950
+Connection ~ 4350 2050
+Wire Wire Line
+	1100 1100 1100 1450
+Wire Wire Line
+	1100 1000 1350 1000
+Wire Wire Line
+	1250 1050 1250 1000
+Connection ~ 1250 1000
+Wire Wire Line
+	1100 1450 2050 1450
+Connection ~ 1250 1450
+Connection ~ 1650 1450
+Wire Wire Line
+	2050 1050 2050 1000
+Connection ~ 2050 1000
+Connection ~ 4350 1050
+Wire Wire Line
+	1950 1000 3650 1000
+Connection ~ 3300 2050
+Connection ~ 3750 2050
 Connection ~ 5800 1350
 Connection ~ 5800 1450
+Wire Wire Line
+	5500 1050 5700 1050
+Wire Wire Line
+	5700 1050 5700 1150
+Wire Wire Line
+	5700 1150 5800 1150
+Wire Wire Line
+	5800 1050 5750 1050
+Wire Wire Line
+	5750 1050 5750 1100
+Wire Wire Line
+	5750 1100 5650 1100
+Wire Wire Line
+	5650 1100 5650 1150
+Wire Wire Line
+	5650 1150 5500 1150
 $EndSCHEMATC
